Commit message: good job

File: urdf/youbot_virtual.urdf (robot description, URDF)
Before this commit: robot youbot, 23 links, 22 joints
Joints:
- joint wheel_joint_bl: limit effort=10 velocity=10 -> lower=-0.5 upper=0.5 effort=10 velocity=10
- joint wheel_joint_br: limit effort=30 velocity=10 -> lower=-0.5 upper=0.5 effort=30 velocity=10
- joint wheel_joint_fl: limit effort=30 velocity=10 -> lower=-0.5 upper=0.5 effort=30 velocity=10
- joint wheel_joint_fr: limit effort=30 velocity=10 -> lower=-0.5 upper=0.5 effort=30 velocity=10
